File: pcb/casing_bottom/casing.kicad_pcb (KiCad board)
At the start: 2 copper layers, 95 x 25 mm, 0 parts

Commit message: PCB MCAD Export
Other:
- outline, holes or cut-outs redrawn
- board text added: "Read Manual Before Use github.com/westonb/little-bee-B1"
- board text removed: "manual and design files at: github.com/westonb/little-bee-B1"
