File: pcb/casing_top/casing.kicad_pcb (KiCad board)
At the start: 2 copper layers, 95 x 25 mm, 1 part

Commit message: PCB MCAD Export
Parts:
- moved G*** 41.9 mm to (147.5, 105.2)
Routing:
- net (no net): track 548.2 -> 1267.5 mm
Other:
- outline, holes or cut-outs redrawn
- board text added: "+B"
- board text added: "+I"
- board text added: "Little Bee B1 Probe Beefield Labs"
- board text removed: "Little Bee B1 Current Probe Beefield Labs"
