File: pcb/current-sense/current-sense.kicad_pcb (KiCad board)
At the start: 4 copper layers, 130 x 25 mm, 108 parts, among them J1 mounting-hole-grounded, J2 mounting-hole-grounded, J3 Tag Connect, J4 mounting-hole-grounded, J5 mounting-hole-grounded, J6 Conn_Coaxial, J7 AA Holder, J8 B2B-XH-A, Q1 FDC6333C, SW1 SW_Push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

Commit message: changes to gain resistors
Parts:
- D4: value B320AF-13 -> NTSAF345T3G
- J1, J2, J4, J5: value mounting-hole-grounded -> M3
- R1, R11, R2, R23, R24, R25, R27, R28: value 4.22k -> 4.7k
- R10: value 2k -> 4.7k
- R16: value 340 -> 470
- R17: value 1.91k -> 1.43k
- R18: value 220 -> 0
- R3, R7: value 121 -> 105
- R38: value 6.81k -> DNP
- R8: value 806 -> 1.43k
Routing:
- net +5V: track 87.7 -> 91.1 mm

Commit message: pre-production PCB assembly
Parts:
- removed TP3: TestPoint, wbraun_smd:THM_COMPACT
- J8: value B2B-XH-A -> DNP
- SW3: footprint Button_Switch_THT:SW_CuK_OS102011MA1QN1_SPDT_Angled -> wbraun_smd:SW_EG1247_SPDT_Angled
Routing:
- net /5V_INT: track 17.5 -> 13.7 mm, vias 3 -> 4
- net /SW1: track 21.3 -> 23.4 mm
- net GNDREF: vias 110 -> 112
- net GND: vias 50 -> 61
- added copper zone on In2.Cu, net /5V_INT
Other:
- board text added: "+"
- board text added: "-"
- board text added: "Gain Adjust"

Commit message: PCB MCAD Export
Parts:
- added REF**: Fiducial_0.5mm_Mask1.5mm, Fiducial:Fiducial_0.5mm_Mask1.5mm, B.Cu at (-8.75, -40.8)
- added REF**: Fiducial_0.5mm_Mask1.5mm, Fiducial:Fiducial_0.5mm_Mask1.5mm, B.Cu at (91.2, -26.8)
- added REF**: Fiducial_0.5mm_Mask1.5mm, Fiducial:Fiducial_0.5mm_Mask1.5mm, B.Cu at (55.5, -47.0)
- added REF**: Fiducial_0.5mm_Mask1.5mm, Fiducial:Fiducial_0.5mm_Mask1.5mm, F.Cu at (-8.75, -40.8)
- added REF**: Fiducial_0.5mm_Mask1.5mm, Fiducial:Fiducial_0.5mm_Mask1.5mm, F.Cu at (56.8, -47.5)
- added REF**: Fiducial_0.5mm_Mask1.5mm, Fiducial:Fiducial_0.5mm_Mask1.5mm, F.Cu at (91.2, -26.8)
- moved G*** 0.35 mm to (83.8, -28.8)
Routing:
- net GNDREF: vias 112 -> 119
Other:
- rule pad_to_mask_clearance: 0.05 -> 0.03
- rule solder_mask_min_width: 0.099 -> 0.07
- board text added: "No mousebite or routing tabs on tip of PCB"
Changed lines of the file:
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@@
   (general
     (thickness 1)
-    (drawings 37)
-    (tracks 1052)
+    (drawings 41)
+    (tracks 1059)
     (zones 0)
-    (modules 107)
+    (modules 113)
     (nets 71)
   )
@@
     (32 B.Adhes user hide)
     (33 F.Adhes user hide)
-    (34 B.Paste user hide)
+    (34 B.Paste user)
     (35 F.Paste user hide)
     (36 B.SilkS user)
@@
     (40 Dwgs.User user)
     (41 Cmts.User user hide)
-    (42 Eco1.User user)
+    (42 Eco1.User user hide)
     (43 Eco2.User user hide)
     (44 Edge.Cuts user)
@@
     (47 F.CrtYd user)
     (48 B.Fab user hide)
-    (49 F.Fab user hide)
+    (49 F.Fab user)
   )
   (setup
-    (last_trace_width 0.16)
+    (last_trace_width 0.127)
     (user_trace_width 0.127)
     (user_trace_width 0.16)
@@
     (mod_text_size 1 1)
     (mod_text_width 0.15)
-    (pad_size 1 1)
+    (pad_size 0.36 0.36)
     (pad_drill 0)
-    (pad_to_mask_clearance 0.05)
-    (solder_mask_min_width 0.099)
+    (pad_to_mask_clearance 0.03)
+    (solder_mask_min_width 0.07)
     (aux_axis_origin 0 0)
     (visible_elements FFF9FF3F)
@@
     (add_net "Net-(U4-Pad5)")
   )
+  (module Fiducial:Fiducial_0.5mm_Mask1.5mm locked (layer B.Cu)
+    (at -8.75 -40.75)
+    (descr "Circular Fiducial, 0.5mm bare copper, 1.5mm soldermask opening")
+    (tags fiducial)
+    (attr smd)
+    (fp_text reference REF** (at 0 1.7145) (layer B.SilkS) hide
+      (effects (font (size 1 1) (thickness 0.15)) (justify mirror))
+    )
+    (fp_text value Fiducial_0.5mm_Mask1.5mm (at 0 -1.7145) (layer B.Fab)
+      (effects (font (size 1 1) (thickness 0.15)) (justify mirror))
+    )
+    (fp_circle (center 0 0) (end 0.75 0) (layer B.Fab) (width 0.1))
+    (fp_circle (center 0 0) (end 1 0) (layer B.CrtYd) (width 0.05))
+    (fp_text user %R (at 0 0) (layer B.Fab) hide
+      (effects (font (size 0.2 0.2) (thickness 0.04)) (justify mirror))
+    )
+    (pad "" smd circle (at 0 0) (size 0.5 0.5) (layers B.Cu B.Mask)
+      (solder_mask_margin 0.5) (clearance 0.5))
+  )
+  (module Fiducial:Fiducial_0.5mm_Mask1.5mm locked (layer B.Cu)
+    (at 91.25 -26.75)
+    (descr "Circular Fiducial, 0.5mm bare copper, 1.5mm soldermask opening")
+    (tags fiducial)
+    (attr smd)
+    (fp_text reference REF** (at 0 1.7145) (layer B.SilkS) hide
+      (effects (font (size 1 1) (thickness 0.15)) (justify mirror))
+    )
+    (fp_text value Fiducial_0.5mm_Mask1.5mm (at 0 -1.7145) (layer B.Fab)
+      (effects (font (size 1 1) (thickness 0.15)) (justify mirror))
+    )
+    (fp_circle (center 0 0) (end 0.75 0) (layer B.Fab) (width 0.1))
+    (fp_circle (center 0 0) (end 1 0) (layer B.CrtYd) (width 0.05))
+    (fp_text user %R (at 0 0) (layer B.Fab) hide
+      (effects (font (size 0.2 0.2) (thickness 0.04)) (justify mirror))
+    )
+    (pad "" smd circle (at 0 0) (size 0.5 0.5) (layers B.Cu B.Mask)
+      (solder_mask_margin 0.5) (clearance 0.5))
+  )
+  (module Fiducial:Fiducial_0.5mm_Mask1.5mm locked (layer B.Cu)
+    (at 55.5 -47)
+    (descr "Circular Fiducial, 0.5mm bare copper, 1.5mm soldermask opening")
+    (tags fiducial)
+    (attr smd)
+    (fp_text reference REF** (at 0 1.7145) (layer B.SilkS) hide
+      (effects (font (size 1 1) (thickness 0.15)) (justify mirror))
+    )
+    (fp_text value Fiducial_0.5mm_Mask1.5mm (at 0 -1.7145) (layer B.Fab)
+      (effects (font (size 1 1) (thickness 0.15)) (justify mirror))
+    )
+    (fp_circle (center 0 0) (end 0.75 0) (layer B.Fab) (width 0.1))
+    (fp_circle (center 0 0) (end 1 0) (layer B.CrtYd) (width 0.05))
+    (fp_text user %R (at 0 0) (layer B.Fab) hide
+      (effects (font (size 0.2 0.2) (thickness 0.04)) (justify mirror))
+    )
+    (pad "" smd circle (at 0 0) (size 0.5 0.5) (layers B.Cu B.Mask)
+      (solder_mask_margin 0.5) (clearance 0.5))
+  )
+  (module Fiducial:Fiducial_0.5mm_Mask1.5mm locked (layer F.Cu)
+    (at -8.75 -40.75)
+    (descr "Circular Fiducial, 0.5mm bare copper, 1.5mm soldermask opening")
+    (tags fiducial)
+    (attr smd)
+    (fp_text reference REF** (at 0 -1.7145) (layer F.SilkS) hide
+      (effects (font (size 1 1) (thickness 0.15)))
+    )
+    (fp_text value Fiducial_0.5mm_Mask1.5mm (at 0 1.7145) (layer F.Fab)
+      (effects (font (size 1 1) (thickness 0.15)))
+    )
+    (fp_circle (center 0 0) (end 0.75 0) (layer F.Fab) (width 0.1))
+    (fp_circle (center 0 0) (end 1 0) (layer F.CrtYd) (width 0.05))
+    (fp_text user %R (at 0 0) (layer F.Fab) hide
+      (effects (font (size 0.2 0.2) (thickness 0.04)))
+    )
+    (pad "" smd circle (at 0 0) (size 0.5 0.5) (layers F.Cu F.Mask)
+      (solder_mask_margin 0.5) (clearance 0.5))
+  )
+  (module Fiducial:Fiducial_0.5mm_Mask1.5mm locked (layer F.Cu)
+    (at 56.75 -47.5)
+    (descr "Circular Fiducial, 0.5mm bare copper, 1.5mm soldermask opening")
+    (tags fiducial)
+    (attr smd)
+    (fp_text reference REF** (at 0 -1.7145) (layer F.SilkS) hide
+      (effects (font (size 1 1) (thickness 0.15)))
+    )
+    (fp_text value Fiducial_0.5mm_Mask1.5mm (at 0 1.7145) (layer F.Fab)
+      (effects (font (size 1 1) (thickness 0.15)))
+    )
+    (fp_circle (center 0 0) (end 0.75 0) (layer F.Fab) (width 0.1))
+    (fp_circle (center 0 0) (end 1 0) (layer F.CrtYd) (width 0.05))
+    (fp_text user %R (at 0 0) (layer F.Fab) hide
+      (effects (font (size 0.2 0.2) (thickness 0.04)))
+    )
+    (pad "" smd circle (at 0 0) (size 0.5 0.5) (layers F.Cu F.Mask)
+      (solder_mask_margin 0.5) (clearance 0.5))
+  )
+  (module Fiducial:Fiducial_0.5mm_Mask1.5mm locked (layer F.Cu)
+    (at 91.25 -26.75)
+    (descr "Circular Fiducial, 0.5mm bare copper, 1.5mm soldermask opening")
+    (tags fiducial)
+    (attr smd)
+    (fp_text reference REF** (at 0 -1.7145) (layer F.SilkS) hide
+      (effects (font (size 1 1) (thickness 0.15)))
+    )
+    (fp_text value Fiducial_0.5mm_Mask1.5mm (at 0 1.7145) (layer F.Fab)
+      (effects (font (size 1 1) (thickness 0.15)))
+    )
+    (fp_circle (center 0 0) (end 0.75 0) (layer F.Fab) (width 0.1))
+    (fp_circle (center 0 0) (end 1 0) (layer F.CrtYd) (width 0.05))
+    (fp_text user %R (at 0 0) (layer F.Fab) hide
+      (effects (font (size 0.2 0.2) (thickness 0.04)))
+    )
+    (pad "" smd circle (at 0 0) (size 0.5 0.5) (layers F.Cu F.Mask)
+      (solder_mask_margin 0.5) (clearance 0.5))
+  )
   (module wbraun_smd:SW_EG1247_SPDT_Angled locked (layer B.Cu)
     (at 74.5 -47.5)
@@
     )
     (fp_poly (pts (xy 0.5 -0.18) (xy -0.5 -0.18) (xy -0.5 0.18) (xy 0.5 0.18)) (layer B.Cu) (width 0))
-    (pad 1 smd circle (at 0.5 0 90) (size 0.36 0.36) (layers B.Cu B.Paste B.Mask)
+    (pad 1 smd circle (at 0.5 0 90) (size 0.36 0.36) (layers B.Cu)
       (net 46 "Net-(J7-Pad2)"))
-    (pad 2 smd circle (at -0.5 0 90) (size 0.36 0.36) (layers B.Cu B.Paste B.Mask)
+    (pad 2 smd circle (at -0.5 0 90) (size 0.36 0.36) (layers B.Cu)
       (net 1 GND))
   )
@@
   )
   (module wbraun_smd:bee_v4 locked (layer F.Cu)
-    (at 83.5 -29)
+    (at 83.75 -28.75)
     (fp_text reference G*** (at 0 0) (layer F.SilkS) hide
       (effects (font (size 1.524 1.524) (thickness 0.3)))
@@
     )
   )
+  (gr_text "No mousebite or routing tabs on tip of PCB" (at -32.65 -46.65) (layer Dwgs.User)
+    (effects (font (size 1 1) (thickness 0.15)))
+  )
+  (gr_text "No mousebite or routing tabs on tip of PCB" (at -32.35 -44.8) (layer Cmts.User)
+    (effects (font (size 1 1) (thickness 0.15)))
+  )
+  (gr_text "No mousebite or routing tabs on tip of PCB" (at -32.55 -43.05) (layer Eco1.User)
+    (effects (font (size 1 1) (thickness 0.15)))
+  )
+  (gr_text "No mousebite or routing tabs on tip of PCB" (at -32.75 -41.65) (layer F.Fab)
+    (effects (font (size 1 1) (thickness 0.15)))
+  )
   (gr_text - (at 18 -49) (layer F.SilkS)
     (effects (font (size 0.8 0.8) (thickness 0.16)))
@@
   (via (at 34.5 -36.7) (size 0.6) (drill 0.3) (layers F.Cu B.Cu) (net 3))
   (via (at 28.3 -46.45) (size 0.6) (drill 0.3) (layers F.Cu B.Cu) (net 3))
+  (via (at 8.25 -33.75) (size 0.6) (drill 0.3) (layers F.Cu B.Cu) (net 3))
+  (via (at 8.25 -40.5) (size 0.6) (drill 0.3) (layers F.Cu B.Cu) (net 3))
+  (via (at -3.25 -39) (size 0.6) (drill 0.3) (layers F.Cu B.Cu) (net 3))
+  (via (at 2.75 -39.25) (size 0.6) (drill 0.3) (layers F.Cu B.Cu) (net 3))
+  (via (at -3.25 -35.25) (size 0.6) (drill 0.3) (layers F.Cu B.Cu) (net 3))
+  (via (at 2.75 -35.5) (size 0.6) (drill 0.3) (layers F.Cu B.Cu) (net 3))
+  (via (at -8.75 -35.25) (size 0.6) (drill 0.3) (layers F.Cu B.Cu) (net 3))
   (segment (start 17.5 -27.9625) (end 17.7125 -27.9625) (width 0.24) (layer F.Cu) (net 4))
   (segment (start 21.44 -29.45) (end 22.15 -29.45) (width 0.24) (layer F.Cu) (net 4))

Commit message: production PCB version
Parts:
- C36: value 1u -> DNP
- Q1: value FDC6333C -> FDC6327C
- R12, R15, R19, R9: value 2k -> 1.43k
- R29: value 102k -> DNP
Routing:
- net +5V: track 91.1 -> 112.0 mm
- net GND: track 83.6 -> 82.8 mm, vias 61 -> 65
- net Net-(J6-Pad1): track 81.9 -> 82.4 mm
- net GNDREF: vias 119 -> 124
Other:
- board text added: "1mm thick PCB No mousebite or routing tabs on tip of PCB"
