File: pcb/current-sense/current-sense.sch (KiCad schematic (older format))
At the start: 107 parts, among them J1 M3, J2 M3, J3 Tag Connect, J4 M3, J5 M3, J6 Conn_Coaxial, J7 AA Holder, J8 B2B-XH-A, Q1 FDC6333C, SW1 SW_Push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

Commit message: changes to gain resistors
Parts:
- R16: value 340 -> 470; MPN RC0603FR-07340RL -> RC0603FR-07470RL
- R17: value 1.91k -> 1.43k; MPN RC0603FR-071K91L -> RC0603FR-071K43L
- R18: value 220 -> 0; MPN RC0603FR-07220RL -> RC0603JR-070RL
- R3, R7: value 121 -> 105; MPN RC0603FR-07121RL -> RC0603FR-07105RL
- R38: value 6.81k -> DNP; MPN RC0603FR-076K81L -> (none)
- R8: value 806 -> 1.43k; MPN RC0603FR-07806RL -> RC0603FR-071K43L
Other:
- note added: "Gain of 1.006\nGain of 4.049"
- note added: "PIC Opamps"
- note added: "Sensor reads 7.3mV/G - 11.42mV/G\nThis includes self heating (50C nominal)\nFlux concentrator is 1.32G/A typical (+-20% ?)\nGain of 32.4 - 13.8 V/V\nGain of 21.14 nominal\n"
- note removed: "Gain of 1.66\nGain of 6.64"
- note removed: "Sensor reads 7.3mV/G - 11.42mV/G\nThis includes self heating (50C nominal)\nFlux concentrator is 1.32G/A typical (+-20% ?)\nGain of 19.5 - 8.3 V/V\nGain of 12.5 nominal\n"
Changed lines of the file:
@@
 P 2150 7600
 F 0 "R7" V 1943 7600 50  0000 C CNN
-F 1 "121" V 2034 7600 50  0000 C CNN
+F 1 "105" V 2034 7600 50  0000 C CNN
 F 2 "Resistor_SMD:R_0603_1608Metric" V 2080 7600 50  0001 C CNN
 F 3 "~" H 2150 7600 50  0001 C CNN
-F 4 "RC0603FR-07121RL" H 2150 7600 50  0001 C CNN "MPN"
+F 4 "RC0603FR-07105RL" H 2150 7600 50  0001 C CNN "MPN"
 	1    2150 7600
 	0    1    1    0
@@
 P 2750 7600
 F 0 "R8" V 2543 7600 50  0000 C CNN
-F 1 "806" V 2634 7600 50  0000 C CNN
+F 1 "1.43k" V 2634 7600 50  0000 C CNN
 F 2 "Resistor_SMD:R_0603_1608Metric" V 2680 7600 50  0001 C CNN
 F 3 "~" H 2750 7600 50  0001 C CNN
-F 4 "RC0603FR-07806RL" H 2750 7600 50  0001 C CNN "MPN"
+F 4 "RC0603FR-071K43L" H 2750 7600 50  0001 C CNN "MPN"
 	1    2750 7600
 	0    1    1    0
@@
 P 1250 7200
 F 0 "R3" H 1180 7154 50  0000 R CNN
-F 1 "121" H 1180 7245 50  0000 R CNN
+F 1 "105" H 1180 7245 50  0000 R CNN
 F 2 "Resistor_SMD:R_0603_1608Metric" V 1180 7200 50  0001 C CNN
 F 3 "~" H 1250 7200 50  0001 C CNN
-F 4 "RC0603FR-07121RL" H 1250 7200 50  0001 C CNN "MPN"
+F 4 "RC0603FR-07105RL" H 1250 7200 50  0001 C CNN "MPN"
 	1    1250 7200
 	-1   0    0    1
@@
 P 6850 7400
 F 0 "R17" V 6643 7400 50  0000 C CNN
-F 1 "1.91k" V 6734 7400 50  0000 C CNN
+F 1 "1.43k" V 6734 7400 50  0000 C CNN
 F 2 "Resistor_SMD:R_0603_1608Metric" V 6780 7400 50  0001 C CNN
 F 3 "~" H 6850 7400 50  0001 C CNN
-F 4 "RC0603FR-071K91L" H 6850 7400 50  0001 C CNN "MPN"
+F 4 "RC0603FR-071K43L" H 6850 7400 50  0001 C CNN "MPN"
 	1    6850 7400
 	0    1    1    0
@@
 P 6850 7850
 F 0 "R18" V 6643 7850 50  0000 C CNN
-F 1 "220" V 6734 7850 50  0000 C CNN
+F 1 "0" V 6734 7850 50  0000 C CNN
 F 2 "Resistor_SMD:R_0603_1608Metric" V 6780 7850 50  0001 C CNN
 F 3 "~" H 6850 7850 50  0001 C CNN
-F 4 "RC0603FR-07220RL" H 6850 7850 50  0001 C CNN "MPN"
+F 4 "RC0603JR-070RL" H 6850 7850 50  0001 C CNN "MPN"
 	1    6850 7850
 	0    1    1    0
@@
 P 6350 7850
 F 0 "R16" V 6143 7850 50  0000 C CNN
-F 1 "340" V 6234 7850 50  0000 C CNN
+F 1 "470" V 6234 7850 50  0000 C CNN
 F 2 "Resistor_SMD:R_0603_1608Metric" V 6280 7850 50  0001 C CNN
 F 3 "~" H 6350 7850 50  0001 C CNN
-F 4 "RC0603FR-07340RL" H 6350 7850 50  0001 C CNN "MPN"
+F 4 "RC0603FR-07470RL" H 6350 7850 50  0001 C CNN "MPN"
 	1    6350 7850
 	0    1    1    0
@@
 $EndComp
 Text Notes 6200 8400 0    50   ~ 0
-Gain of 1.66\nGain of 6.64
+Gain of 1.006\nGain of 4.049
 Wire Wire Line
 	1250 7550 1600 7550
@@
 P 3150 8050
 F 0 "R38" V 3357 8050 50  0000 C CNN
-F 1 "6.81k" V 3266 8050 50  0000 C CNN
+F 1 "DNP" V 3266 8050 50  0000 C CNN
 F 2 "Resistor_SMD:R_0603_1608Metric" V 3080 8050 50  0001 C CNN
 F 3 "~" H 3150 8050 50  0001 C CNN
-F 4 "RC0603FR-076K81L" H 3150 8050 50  0001 C CNN "MPN"
+F 4 "" H 3150 8050 50  0001 C CNN "MPN"
 	1    3150 8050
 	0    -1   -1   0
@@
 	10400 4350 10800 4350
 Text Notes 1100 8900 0    50   ~ 0
-Sensor reads  7.3mV/G - 11.42mV/G\nThis includes self heating (50C nominal)\nFlux concentrator is 1.32G/A typical (+-20% ?)\nGain of 19.5 - 8.3 V/V\nGain of 12.5 nominal\n
+Sensor reads  7.3mV/G - 11.42mV/G\nThis includes self heating (50C nominal)\nFlux concentrator is 1.32G/A typical (+-20% ?)\nGain of 32.4 - 13.8 V/V\nGain of 21.14 nominal\n
 $Comp
 L Device:C C36
@@
 	1    0    0    -1
 $EndComp
+Text Notes 5350 5450 0    50   ~ 0
+PIC Opamps
 $EndSCHEMATC

Commit message: pre-production PCB assembly
Parts:
- removed TP3: TestPoint, wbraun_smd:THM_COMPACT, symbol Connector:TestPoint
- J8: value B2B-XH-A -> DNP
- SW3: footprint Button_Switch_THT:SW_CuK_OS102011MA1QN1_SPDT_Angled -> wbraun_smd:SW_EG1247_SPDT_Angled; symbol Switch:SW_SPDT -> wbraun_ic_lib:SW_SPDT_w_MP
Connections:
- wire segments 395 -> 396
Changed lines of the file:
@@
 	0    1    1    0
 $EndComp
-$Comp
-L Connector:TestPoint TP3
-U 1 1 5EF26D62
-P 7100 2350
-F 0 "TP3" H 7042 2377 50  0000 R CNN
-F 1 "TestPoint" H 7150 2000 50  0000 R CNN
-F 2 "wbraun_smd:THM_COMPACT" H 7300 2350 50  0001 C CNN
-F 3 "~" H 7300 2350 50  0001 C CNN
-	1    7100 2350
-	1    0    0    -1
-$EndComp
-$Comp
-L power:GND #PWR025
-U 1 1 5EF26FD0
-P 7100 2400
-F 0 "#PWR025" H 7100 2150 50  0001 C CNN
-F 1 "GND" H 7105 2227 50  0000 C CNN
-F 2 "" H 7100 2400 50  0001 C CNN
-F 3 "" H 7100 2400 50  0001 C CNN
-	1    7100 2400
-	1    0    0    -1
-$EndComp
-Wire Wire Line
-	7100 2350 7100 2400
 Text Label 2300 4200 0    50   ~ 0
 SR
@@
 P 8450 4650
 F 0 "J8" H 8342 4325 50  0000 C CNN
-F 1 "B2B-XH-A" H 8342 4416 50  0000 C CNN
+F 1 "DNP" H 8342 4416 50  0000 C CNN
 F 2 "Connector_JST:JST_XH_B2B-XH-A_1x02_P2.50mm_Vertical" H 8450 4650 50  0001 C CNN
 F 3 "~" H 8450 4650 50  0001 C CNN
@@
 5V_INT
 $Comp
-L Switch:SW_SPDT SW3
+L wbraun_ic_lib:SW_SPDT_w_MP SW3
 U 1 1 5EF02AA2
 P 10800 3350
 F 0 "SW3" H 10850 3150 50  0000 C CNN
 F 1 "SW_SPDT" H 10850 3050 50  0000 C CNN
-F 2 "Button_Switch_THT:SW_CuK_OS102011MA1QN1_SPDT_Angled" H 10800 3350 50  0001 C CNN
+F 2 "wbraun_smd:SW_EG1247_SPDT_Angled" H 10800 3350 50  0001 C CNN
 F 3 "~" H 10800 3350 50  0001 C CNN
 F 4 "EG1247" H 2600 2450 50  0001 C CNN "MPN"
@@
 Text Notes 5350 5450 0    50   ~ 0
 PIC Opamps
+$Comp
+L power:GND #PWR0137
+U 1 1 601DCBB5
+P 10550 3600
+F 0 "#PWR0137" H 10550 3350 50  0001 C CNN
+F 1 "GND" H 10555 3427 50  0000 C CNN
+F 2 "" H 10550 3600 50  0001 C CNN
+F 3 "" H 10550 3600 50  0001 C CNN
+	1    10550 3600
+	1    0    0    -1
+$EndComp
+Wire Wire Line
+	10600 3450 10550 3450
+Wire Wire Line
+	10550 3450 10550 3600
 $EndSCHEMATC

Commit message: PCB MCAD Export
Connections:
- no-connect marks 0 -> 4
Changed lines of the file:
@@
 Wire Wire Line
 	10550 3450 10550 3600
+NoConn ~ 3450 1300
+NoConn ~ 4750 1300
+NoConn ~ 11000 3250
+NoConn ~ 2200 4050
+$Comp
+L power:PWR_FLAG #FLG0101
+U 1 1 603BE599
+P 10800 4300
+F 0 "#FLG0101" H 10800 4375 50  0001 C CNN
+F 1 "PWR_FLAG" H 10800 4473 50  0000 C CNN
+F 2 "" H 10800 4300 50  0001 C CNN
+F 3 "~" H 10800 4300 50  0001 C CNN
+	1    10800 4300
+	1    0    0    -1
+$EndComp
+Wire Wire Line
+	10800 4300 10800 4350
+Connection ~ 10800 4350
+$Comp
+L power:PWR_FLAG #FLG0102
+U 1 1 603EB5A9
+P 11100 5950
+F 0 "#FLG0102" H 11100 6025 50  0001 C CNN
+F 1 "PWR_FLAG" H 11100 6123 50  0000 C CNN
+F 2 "" H 11100 5950 50  0001 C CNN
+F 3 "~" H 11100 5950 50  0001 C CNN
+	1    11100 5950
+	1    0    0    -1
+$EndComp
+$Comp
+L power:GND #PWR0138
+U 1 1 603EB866
+P 11100 6100
+F 0 "#PWR0138" H 11100 5850 50  0001 C CNN
+F 1 "GND" H 11105 5927 50  0000 C CNN
+F 2 "" H 11100 6100 50  0001 C CNN
+F 3 "" H 11100 6100 50  0001 C CNN
+	1    11100 6100
+	1    0    0    -1
+$EndComp
+Wire Wire Line
+	11100 6100 11100 5950
+$Comp
+L power:+5V #PWR0139
+U 1 1 604164F4
+P 11500 6100
+F 0 "#PWR0139" H 11500 5950 50  0001 C CNN
+F 1 "+5V" H 11515 6273 50  0000 C CNN
+F 2 "" H 11500 6100 50  0001 C CNN
+F 3 "" H 11500 6100 50  0001 C CNN
+	1    11500 6100
+	-1   0    0    1
+$EndComp
+Wire Wire Line
+	11500 5950 11500 6100
+$Comp
+L power:GNDREF #PWR0140
+U 1 1 604425CA
+P 11950 6150
+F 0 "#PWR0140" H 11950 5900 50  0001 C CNN
+F 1 "GNDREF" H 11955 5977 50  0000 C CNN
+F 2 "" H 11950 6150 50  0001 C CNN
+F 3 "" H 11950 6150 50  0001 C CNN
+	1    11950 6150
+	1    0    0    -1
+$EndComp
+$Comp
+L power:PWR_FLAG #FLG0103
+U 1 1 60444269
+P 11500 5950
+F 0 "#FLG0103" H 11500 6025 50  0001 C CNN
+F 1 "PWR_FLAG" H 11500 6123 50  0000 C CNN
+F 2 "" H 11500 5950 50  0001 C CNN
+F 3 "~" H 11500 5950 50  0001 C CNN
+	1    11500 5950
+	1    0    0    -1
+$EndComp
+$Comp
+L power:PWR_FLAG #FLG0104
+U 1 1 60444653
+P 11950 5950
+F 0 "#FLG0104" H 11950 6025 50  0001 C CNN
+F 1 "PWR_FLAG" H 11950 6123 50  0000 C CNN
+F 2 "" H 11950 5950 50  0001 C CNN
+F 3 "~" H 11950 5950 50  0001 C CNN
+	1    11950 5950
+	1    0    0    -1
+$EndComp
+Wire Wire Line
+	11950 5950 11950 6150
 $EndSCHEMATC

Commit message: production PCB version
Parts:
- C10, C11, C12, C15, C16, C19, C2, C23, C25, C26, C27, C28, C29, C3, C30, C31, C32, C34, C5, C8, C9: MPN CL10A105KO8NNNC -> CL10B105KO8NNNC
- C36: value 1u -> DNP; MPN CL10A105KO8NNNC -> (none)
- Q1: value FDC6333C -> FDC6327C; MPN FDC6333C -> FDC6327C
- R12, R15, R19, R9: value 2k -> 1.43k; MPN RC0603FR-072KL -> RC0603FR-071K43L
- R21: MPN RC0603FR-07102KL -> RMCF0603FT102K
- R29: value 102k -> DNP; MPN RC0603FR-07102KL -> (none)
Changed lines of the file:
@@
 P 1500 2200
 F 0 "Q1" H 1600 2200 50  0000 L CNN
-F 1 "FDC6333C" H 1600 2100 50  0000 L CNN
+F 1 "FDC6327C" H 1600 2100 50  0000 L CNN
 F 2 "Package_TO_SOT_SMD:TSOT-23-6" H 1450 1725 50  0001 C CNN
-F 3 "https://www.diodes.com/assets/Datasheets/DMC2053UVT.pdf" H 1400 2200 50  0001 C CNN
-F 4 "FDC6333C" H 0   500 50  0001 C CNN "MPN"
+F 3 "" H 1400 2200 50  0001 C CNN
+F 4 "FDC6327C" H 0   500 50  0001 C CNN "MPN"
 	1    1500 2200
 	1    0    0    -1
@@
 P 1500 1700
 F 0 "Q1" H 1600 1650 50  0000 L CNN
-F 1 "FDC6333C" H 1600 1550 50  0000 L CNN
+F 1 "FDC6327C" H 1600 1550 50  0000 L CNN
 F 2 "Package_TO_SOT_SMD:TSOT-23-6" H 1450 1225 50  0001 C CNN
-F 3 "https://www.diodes.com/assets/Datasheets/DMC2053UVT.pdf" H 1400 1700 50  0001 C CNN
-F 4 "FDC6333C" H 0   -500 50  0001 C CNN "MPN"
+F 3 "" H 1400 1700 50  0001 C CNN
+F 4 "FDC6327C" H 0   -500 50  0001 C CNN "MPN"
 	2    1500 1700
 	1    0    0    1
@@
 F 2 "Capacitor_SMD:C_0603_1608Metric" H 2038 1800 50  0001 C CNN
 F 3 "~" H 2000 1950 50  0001 C CNN
-F 4 "CL10A105KO8NNNC" H 0   0   50  0001 C CNN "MPN"
+F 4 "CL10B105KO8NNNC" H 0   0   50  0001 C CNN "MPN"
 	1    2000 1950
 	0    -1   -1   0
@@
 F 2 "Capacitor_SMD:C_0603_1608Metric" H 12838 6950 50  0001 C CNN
 F 3 "~" H 12800 7100 50  0001 C CNN
-F 4 "CL10A105KO8NNNC" H 4950 4250 50  0001 C CNN "MPN"
+F 4 "CL10B105KO8NNNC" H 4950 4250 50  0001 C CNN "MPN"
 	1    12800 7100
 	1    0    0    -1
@@
 F 2 "Capacitor_SMD:C_0603_1608Metric" H 4138 2400 50  0001 C CNN
 F 3 "~" H 4100 2550 50  0001 C CNN
-F 4 "CL10A105KO8NNNC" H 0   0   50  0001 C CNN "MPN"
+F 4 "CL10B105KO8NNNC" H 0   0   50  0001 C CNN "MPN"
 	1    4100 2550
 	1    0    0    -1
@@
 P 6450 5000
 F 0 "R15" V 6657 5000 50  0000 C CNN
-F 1 "2k" V 6566 5000 50  0000 C CNN
+F 1 "1.43k" V 6566 5000 50  0000 C CNN
 F 2 "Resistor_SMD:R_0603_1608Metric" V 6380 5000 50  0001 C CNN
 F 3 "~" H 6450 5000 50  0001 C CNN
-F 4 "RC0603FR-072KL" H -750 1200 50  0001 C CNN "MPN"
+F 4 "RC0603FR-071K43L" H -750 1200 50  0001 C CNN "MPN"
 	1    6450 5000
 	0    -1   -1   0
@@
 F 2 "Capacitor_SMD:C_0603_1608Metric" H 6788 5100 50  0001 C CNN
 F 3 "~" H 6750 5250 50  0001 C CNN
-F 4 "CL10A105KO8NNNC" H -750 1200 50  0001 C CNN "MPN"
+F 4 "CL10B105KO8NNNC" H -750 1200 50  0001 C CNN "MPN"
 	1    6750 5250
 	1    0    0    -1
@@
 F 2 "Capacitor_SMD:C_0603_1608Metric" H 12988 8100 50  0001 C CNN
 F 3 "~" H 12950 8250 50  0001 C CNN
-F 4 "CL10A105KO8NNNC" H 3550 2600 50  0001 C CNN "MPN"
+F 4 "CL10B105KO8NNNC" H 3550 2600 50  0001 C CNN "MPN"
 	1    12950 8250
 	1    0    0    -1
@@
 F 2 "Capacitor_SMD:C_0603_1608Metric" H 12988 8500 50  0001 C CNN
 F 3 "~" H 12950 8650 50  0001 C CNN
-F 4 "CL10A105KO8NNNC" H 3550 2600 50  0001 C CNN "MPN"
+F 4 "CL10B105KO8NNNC" H 3550 2600 50  0001 C CNN "MPN"
 	1    12950 8650
 	1    0    0    -1
@@
 F 2 "Capacitor_SMD:C_0603_1608Metric" H 14838 8300 50  0001 C CNN
 F 3 "~" H 14800 8450 50  0001 C CNN
-F 4 "CL10A105KO8NNNC" H 4400 2600 50  0001 C CNN "MPN"
+F 4 "CL10B105KO8NNNC" H 4400 2600 50  0001 C CNN "MPN"
 	1    14800 8450
 	1    0    0    -1
@@
 P 4350 850
 F 0 "R12" V 4557 850 50  0000 C CNN
-F 1 "2k" V 4466 850 50  0000 C CNN
+F 1 "1.43k" V 4466 850 50  0000 C CNN
 F 2 "Resistor_SMD:R_0603_1608Metric" V 4280 850 50  0001 C CNN
 F 3 "~" H 4350 850 50  0001 C CNN
-F 4 "RC0603FR-072KL" H 4350 850 50  0001 C CNN "MPN"
+F 4 "RC0603FR-071K43L" H 4350 850 50  0001 C CNN "MPN"
 	1    4350 850
 	0    -1   -1   0
@@
 F 2 "Capacitor_SMD:C_0603_1608Metric" H 14338 8300 50  0001 C CNN
 F 3 "~" H 14300 8450 50  0001 C CNN
-F 4 "CL10A105KO8NNNC" H 3900 2600 50  0001 C CNN "MPN"
+F 4 "CL10B105KO8NNNC" H 3900 2600 50  0001 C CNN "MPN"
 	1    14300 8450
 	1    0    0    -1
@@
 F 2 "Resistor_SMD:R_0603_1608Metric" V 13430 5150 50  0001 C CNN
 F 3 "~" H 13500 5150 50  0001 C CNN
-F 4 "RC0603FR-07102KL" H 13500 5150 50  0001 C CNN "MPN"
+F 4 "RMCF0603FT102K" H 13500 5150 50  0001 C CNN "MPN"
 	1    13500 5150
 	1    0    0    -1
@@
 F 2 "Capacitor_SMD:C_0603_1608Metric" H 1638 7050 50  0001 C CNN
 F 3 "~" H 1600 7200 50  0001 C CNN
-F 4 "CL10A105KO8NNNC" H 1600 7200 50  0001 C CNN "MPN"
+F 4 "CL10B105KO8NNNC" H 1600 7200 50  0001 C CNN "MPN"
 	1    1600 7200
 	1    0    0    -1
@@
 P 3400 6400
 F 0 "R9" H 3330 6354 50  0000 R CNN
-F 1 "2k" H 3330 6445 50  0000 R CNN
+F 1 "1.43k" H 3330 6445 50  0000 R CNN
 F 2 "Resistor_SMD:R_0603_1608Metric" V 3330 6400 50  0001 C CNN
 F 3 "~" H 3400 6400 50  0001 C CNN
-F 4 "RC0603FR-072KL" H 3400 6400 50  0001 C CNN "MPN"
+F 4 "RC0603FR-071K43L" H 3400 6400 50  0001 C CNN "MPN"
 	1    3400 6400
 	-1   0    0    1
@@
 P 8350 6450
 F 0 "R19" H 8280 6404 50  0000 R CNN
-F 1 "2k" H 8280 6495 50  0000 R CNN
+F 1 "1.43k" H 8280 6495 50  0000 R CNN
 F 2 "Resistor_SMD:R_0603_1608Metric" V 8280 6450 50  0001 C CNN
 F 3 "~" H 8350 6450 50  0001 C CNN
-F 4 "RC0603FR-072KL" H 8350 6450 50  0001 C CNN "MPN"
+F 4 "RC0603FR-071K43L" H 8350 6450 50  0001 C CNN "MPN"
 	1    8350 6450
 	-1   0    0    1
@@
 F 2 "Capacitor_SMD:C_0603_1608Metric" H 13438 8100 50  0001 C CNN
 F 3 "~" H 13400 8250 50  0001 C CNN
-F 4 "CL10A105KO8NNNC" H 4000 2600 50  0001 C CNN "MPN"
+F 4 "CL10B105KO8NNNC" H 4000 2600 50  0001 C CNN "MPN"
 	1    13400 8250
 	1    0    0    -1
@@
 F 2 "Capacitor_SMD:C_0603_1608Metric" H 13438 8500 50  0001 C CNN
 F 3 "~" H 13400 8650 50  0001 C CNN
-F 4 "CL10A105KO8NNNC" H 4000 2600 50  0001 C CNN "MPN"
+F 4 "CL10B105KO8NNNC" H 4000 2600 50  0001 C CNN "MPN"
 	1    13400 8650
 	1    0    0    -1
@@
 P 12350 4200
 F 0 "R29" H 12420 4246 50  0000 L CNN
-F 1 "102k" H 12420 4155 50  0000 L CNN
+F 1 "DNP" H 12420 4155 50  0000 L CNN
 F 2 "Resistor_SMD:R_0603_1608Metric" V 12280 4200 50  0001 C CNN
 F 3 "~" H 12350 4200 50  0001 C CNN
-F 4 "RC0603FR-07102KL" H 2350 -350 50  0001 C CNN "MPN"
+F 4 "" H 2350 -350 50  0001 C CNN "MPN"
 	1    12350 4200
 	1    0    0    -1
@@
 F 2 "Capacitor_SMD:C_0603_1608Metric" H 6838 3900 50  0001 C CNN
 F 3 "~" H 6800 4050 50  0001 C CNN
-F 4 "CL10A105KO8NNNC" H -700 0   50  0001 C CNN "MPN"
+F 4 "CL10B105KO8NNNC" H -700 0   50  0001 C CNN "MPN"
 	1    6800 4050
 	1    0    0    -1
@@
 F 2 "Capacitor_SMD:C_0603_1608Metric" H 12638 2900 50  0001 C CNN
 F 3 "~" H 12600 3050 50  0001 C CNN
-F 4 "CL10A105KO8NNNC" H 3200 -2600 50  0001 C CNN "MPN"
+F 4 "CL10B105KO8NNNC" H 3200 -2600 50  0001 C CNN "MPN"
 	1    12600 3050
 	0    1    1    0
@@
 F 2 "Capacitor_SMD:C_0603_1608Metric" H 13488 2900 50  0001 C CNN
 F 3 "~" H 13450 3050 50  0001 C CNN
-F 4 "CL10A105KO8NNNC" H 5600 200 50  0001 C CNN "MPN"
+F 4 "CL10B105KO8NNNC" H 5600 200 50  0001 C CNN "MPN"
 	1    13450 3050
 	1    0    0    -1
@@
 F 2 "Capacitor_SMD:C_0603_1608Metric" H 14988 2900 50  0001 C CNN
 F 3 "~" H 14950 3050 50  0001 C CNN
-F 4 "CL10A105KO8NNNC" H 7100 200 50  0001 C CNN "MPN"
+F 4 "CL10B105KO8NNNC" H 7100 200 50  0001 C CNN "MPN"
 	1    14950 3050
 	1    0    0    -1
@@
 F 2 "Capacitor_SMD:C_0603_1608Metric" H 12638 1050 50  0001 C CNN
 F 3 "~" H 12600 1200 50  0001 C CNN
-F 4 "CL10A105KO8NNNC" H 3200 -4450 50  0001 C CNN "MPN"
+F 4 "CL10B105KO8NNNC" H 3200 -4450 50  0001 C CNN "MPN"
 	1    12600 1200
 	0    1    1    0
@@
 F 2 "Capacitor_SMD:C_0603_1608Metric" H 13488 1050 50  0001 C CNN
 F 3 "~" H 13450 1200 50  0001 C CNN
-F 4 "CL10A105KO8NNNC" H 5600 -1650 50  0001 C CNN "MPN"
+F 4 "CL10B105KO8NNNC" H 5600 -1650 50  0001 C CNN "MPN"
 	1    13450 1200
 	1    0    0    -1
@@
 F 2 "Capacitor_SMD:C_0603_1608Metric" H 14988 1050 50  0001 C CNN
 F 3 "~" H 14950 1200 50  0001 C CNN
-F 4 "CL10A105KO8NNNC" H 7100 -1650 50  0001 C CNN "MPN"
+F 4 "CL10B105KO8NNNC" H 7100 -1650 50  0001 C CNN "MPN"
 	1    14950 1200
 	1    0    0    -1
@@
 F 2 "Capacitor_SMD:C_0603_1608Metric" H 1588 4850 50  0001 C CNN
 F 3 "~" H 1550 5000 50  0001 C CNN
-F 4 "CL10A105KO8NNNC" H -6300 2150 50  0001 C CNN "MPN"
+F 4 "CL10B105KO8NNNC" H -6300 2150 50  0001 C CNN "MPN"
 	1    1550 5000
 	-1   0    0    -1
@@
 F 2 "Capacitor_SMD:C_0603_1608Metric" H 2088 4850 50  0001 C CNN
 F 3 "~" H 2050 5000 50  0001 C CNN
-F 4 "CL10A105KO8NNNC" H -5800 2150 50  0001 C CNN "MPN"
+F 4 "CL10B105KO8NNNC" H -5800 2150 50  0001 C CNN "MPN"
 	1    2050 5000
 	-1   0    0    -1
@@
 F 2 "Capacitor_SMD:C_0603_1608Metric" H 13488 1800 50  0001 C CNN
 F 3 "~" H 13450 1950 50  0001 C CNN
-F 4 "CL10A105KO8NNNC" H 5600 -900 50  0001 C CNN "MPN"
+F 4 "CL10B105KO8NNNC" H 5600 -900 50  0001 C CNN "MPN"
 	1    13450 1950
 	1    0    0    -1
@@
 P 12350 3700
 F 0 "C36" H 12465 3746 50  0000 L CNN
-F 1 "1u" H 12465 3655 50  0000 L CNN
+F 1 "DNP" H 12465 3655 50  0000 L CNN
 F 2 "Capacitor_SMD:C_0603_1608Metric" H 12388 3550 50  0001 C CNN
 F 3 "~" H 12350 3700 50  0001 C CNN
-F 4 "CL10A105KO8NNNC" H 4850 -350 50  0001 C CNN "MPN"
+F 4 "" H 4850 -350 50  0001 C CNN "MPN"
 	1    12350 3700
 	1    0    0    -1
